File: hw/ttlcalc2_bypass.kicad_sch (KiCad schematic)
At the start: 35 parts

Commit message: PCB cleanup
Swap location of I/O output register and address latch
Clean up routing
Via stitch around clock traces
Fill out sheet description block
Other:
- title: (none) -> TTL Calculator Logic Board
Changed lines of the file:
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@@
 	(generator_version "8.0")
 	(paper "A4")
+	(title_block
+		(title "TTL Calculator Logic Board")
+		(date "2025-02-12")
+		(rev "B")
+	)
 	(junction
 		(at 60.96 80.01)
