File: hw/ttlcalc2_front/ttlcalc2_front.kicad_pcb (KiCad board)
At the start: 2 copper layers, 330.2 x 76.2 mm, 61 parts, among them J1 DISP_CONN, J2 PWR_HV

Commit message: Minor display hardware revisions
Add anti-ghosting inter-cathode resistors to nixies
Adjust component values based on experiments
Change from individual netclass labels to rule areas
Tweak traces on display board
Update .gitignore to ignore KiCad lock files
Parts:
- added R17: 470k, Resistor_THT:R_Axial_DIN0207_L6.3mm_D2.5mm_P7.62mm_Horizontal, F.Cu at (347.0, 101.0)
- added R18: 470k, Resistor_THT:R_Axial_DIN0207_L6.3mm_D2.5mm_P7.62mm_Horizontal, F.Cu at (342.9, 101.0)
- added R19: 470k, Resistor_THT:R_Axial_DIN0207_L6.3mm_D2.5mm_P7.62mm_Horizontal, F.Cu at (338.9, 101.0)
- added R20: 470k, Resistor_THT:R_Axial_DIN0207_L6.3mm_D2.5mm_P7.62mm_Horizontal, F.Cu at (334.8, 101.0)
- added R21: 470k, Resistor_THT:R_Axial_DIN0207_L6.3mm_D2.5mm_P7.62mm_Horizontal, F.Cu at (330.8, 101.0)
- added R22: 470k, Resistor_THT:R_Axial_DIN0207_L6.3mm_D2.5mm_P7.62mm_Horizontal, F.Cu at (326.7, 101.0)
- added R23: 470k, Resistor_THT:R_Axial_DIN0207_L6.3mm_D2.5mm_P7.62mm_Horizontal, F.Cu at (322.7, 101.0)
- added R24: 470k, Resistor_THT:R_Axial_DIN0207_L6.3mm_D2.5mm_P7.62mm_Horizontal, F.Cu at (318.6, 101.0)
- added R25: 470k, Resistor_THT:R_Axial_DIN0207_L6.3mm_D2.5mm_P7.62mm_Horizontal, F.Cu at (314.6, 101.0)
- added R26: 470k, Resistor_THT:R_Axial_DIN0207_L6.3mm_D2.5mm_P7.62mm_Horizontal, F.Cu at (310.5, 101.0)
- R1, R10, R11, R12, R15, R16, R2, R3, R4, R5, R6, R7, R8, R9: value 470k -> 220k
- R13, R14: value 100k -> 150k
Routing:
- net Net-(R17-Pad2): track 0.00 -> 36.4 mm
- net NXC_2: track 533.3 -> 552.6 mm, vias 15 -> 16
- net NXC_3: track 629.8 -> 647.0 mm, vias 15 -> 16
- net NXC_1: track 473.6 -> 490.6 mm, vias 15 -> 16
- net NXC_4: track 731.9 -> 748.6 mm
- net NXC_5: track 786.9 -> 801.4 mm, vias 14 -> 15
- net NXC_6: track 914.8 -> 928.0 mm, vias 15 -> 16
- net NXC_7: track 846.3 -> 858.3 mm, vias 15 -> 16
- net NXC_8: track 789.3 -> 800.1 mm, vias 15 -> 16
- net NXC_0: track 514.7 -> 525.0 mm, vias 15 -> 16
- net NXC_9: track 747.0 -> 756.2 mm, vias 15 -> 16
- net NE_NEG_E: track 216.6 -> 210.9 mm
- net DP_4: track 80.7 -> 81.2 mm
