File: hw/ttlcalc2_display/ttlcalc2_display.kicad_pcb (KiCad board)
At the start: 2 copper layers, 167.6 x 177.8 mm, 186 parts, among them J1 DISP_CONN, J2 HV_PWR, J3 5V_PWR, J4 IO_BUS, Q1 MPSA42, Q10 MPSA42, Q11 MPSA42, Q12 MPSA42, Q13 MPSA42, Q14 MPSA42, Q15 MPSA42, Q16 MPSA42, Q17 MPSA42, Q18 MPSA42, Q19 MPSA92, Q2 MPSA42, Q20 MPSA92, Q21 MPSA92, Q22 MPSA92, Q23 MPSA92, Q24 MPSA42, Q25 MPSA42, Q26 MPSA42, Q27 MPSA42, Q28 MPSA42, Q29 MPSA42, Q3 MPSA42, Q30 MPSA42, Q31 MPSA42, Q32 MPSA92, Q33 MPSA92, Q34 MPSA92, Q35 MPSA92, Q36 MPSA92, Q37 MPSA92, Q38 MPSA92, Q39 MPSA92, Q4 MPSA42, Q40 MPSA92, Q41 MPSA42, Q42 MPSA42, Q43 MPSA42, Q44 MPSA42, Q45 MPSA42, Q46 MPSA42, Q47 MPSA42, Q48 MPSA42, Q49 MPSA42, Q5 MPSA42, Q50 MPSA42, Q51 MPSA42, Q52 MPSA42, Q53 MPSA42, Q54 MPSA42, Q6 MPSA42, Q7 MPSA42, Q8 MPSA42, Q9 MPSA42, U1 74LS173, U10 74LS138, U11 74LS138, U12 74LS42, U13 74LS04, U14 74LS04, U15 74LS04, U16 74LS138, U17 74LS08, U18 74LS173, U19 74LS173, U2 74LS138, U3 74LS138, U4 74LS173, U5 74LS04, U6 74LS04, U7 74LS04, U8 74LS04, U9 74LS138

Commit message: More resistor value updates, ERC fixes
Update Nixie anode resistors to 22k based on calculation and experimental verification
Fix ERC errors due to remaining Logic netclass labels in decimal point sheet
Parts:
- R1, R10, R11, R12, R13, R14, R2, R3, R4, R5, R6, R7, R8, R9: value 10k -> 22k
Changed lines of the file:
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@@
 			)
 		)
-		(property "Value" "10k"
+		(property "Value" "22k"
 			(at 3.81 0 0)
 			(layer "F.SilkS")
@@
 			)
 		)
-		(property "Value" "10k"
+		(property "Value" "22k"
 			(at 3.81 0 0)
 			(layer "F.SilkS")
@@
 			)
 		)
-		(property "Value" "10k"
+		(property "Value" "22k"
 			(at 3.81 0 0)
 			(layer "F.SilkS")
@@
 			)
 		)
-		(property "Value" "10k"
+		(property "Value" "22k"
 			(at 3.81 0 0)
 			(layer "F.SilkS")
@@
 			)
 		)
-		(property "Value" "10k"
+		(property "Value" "22k"
 			(at 3.81 0 0)
 			(layer "F.SilkS")
@@
 			)
 		)
-		(property "Value" "10k"
+		(property "Value" "22k"
 			(at 3.81 0 0)
 			(layer "F.SilkS")
@@
 			)
 		)
-		(property "Value" "10k"
+		(property "Value" "22k"
 			(at 3.81 0 0)
 			(layer "F.SilkS")
@@
 			)
 		)
-		(property "Value" "10k"
+		(property "Value" "22k"
 			(at 3.81 0 0)
 			(layer "F.SilkS")
@@
 			)
 		)
-		(property "Value" "10k"
+		(property "Value" "22k"
 			(at 3.81 0 0)
 			(layer "F.SilkS")
@@
 			)
 		)
-		(property "Value" "10k"
+		(property "Value" "22k"
 			(at 3.81 0 0)
 			(layer "F.SilkS")
@@
 			)
 		)
-		(property "Value" "10k"
+		(property "Value" "22k"
 			(at 3.81 0 0)
 			(layer "F.SilkS")
@@
 			)
 		)
-		(property "Value" "10k"
+		(property "Value" "22k"
 			(at 3.81 0 0)
 			(layer "F.SilkS")
@@
 			)
 		)
-		(property "Value" "10k"
+		(property "Value" "22k"
 			(at 3.81 0 0)
 			(layer "F.SilkS")
@@
 			)
 		)
-		(property "Value" "10k"
+		(property "Value" "22k"
 			(at 3.81 0 0)
 			(layer "F.SilkS")
