File: hw/ttlcalc2_display/ttlcalc2_display_dps.kicad_sch (KiCad schematic)
At the start: 32 parts, among them Q10 MPSA42, Q11 MPSA42, Q4 MPSA42, Q5 MPSA42, Q6 MPSA42, Q7 MPSA42, Q8 MPSA42, Q9 MPSA42, U10 74LS138, U11 74LS04, U8 74LS04, U9 74LS138

Commit message: Continue work on display driver board schematic
Parts:
- R10: renamed from R12; footprint Resistor_THT:R_Axial_DIN0309_L9.0mm_D3.2mm_P2.54mm_Vertical -> Resistor_THT:R_Axial_DIN0207_L6.3mm_D2.5mm_P2.54mm_Vertical
- R11: renamed from R13; footprint Resistor_THT:R_Axial_DIN0309_L9.0mm_D3.2mm_P2.54mm_Vertical -> Resistor_THT:R_Axial_DIN0207_L6.3mm_D2.5mm_P2.54mm_Vertical
- R12: renamed from R7; footprint Resistor_THT:R_Axial_DIN0309_L9.0mm_D3.2mm_P2.54mm_Vertical -> Resistor_THT:R_Axial_DIN0207_L6.3mm_D2.5mm_P2.54mm_Vertical
- R13: renamed from R8; footprint Resistor_THT:R_Axial_DIN0309_L9.0mm_D3.2mm_P2.54mm_Vertical -> Resistor_THT:R_Axial_DIN0207_L6.3mm_D2.5mm_P2.54mm_Vertical
- R14, R15, R16, R17: renamed from R?; footprint Resistor_THT:R_Axial_DIN0309_L9.0mm_D3.2mm_P2.54mm_Vertical -> Resistor_THT:R_Axial_DIN0207_L6.3mm_D2.5mm_P2.54mm_Vertical
- R6: footprint Resistor_THT:R_Axial_DIN0309_L9.0mm_D3.2mm_P2.54mm_Vertical -> Resistor_THT:R_Axial_DIN0207_L6.3mm_D2.5mm_P2.54mm_Vertical
- R7: renamed from R9; footprint Resistor_THT:R_Axial_DIN0309_L9.0mm_D3.2mm_P2.54mm_Vertical -> Resistor_THT:R_Axial_DIN0207_L6.3mm_D2.5mm_P2.54mm_Vertical
- R8: renamed from R10; footprint Resistor_THT:R_Axial_DIN0309_L9.0mm_D3.2mm_P2.54mm_Vertical -> Resistor_THT:R_Axial_DIN0207_L6.3mm_D2.5mm_P2.54mm_Vertical
- R9: renamed from R11; footprint Resistor_THT:R_Axial_DIN0309_L9.0mm_D3.2mm_P2.54mm_Vertical -> Resistor_THT:R_Axial_DIN0207_L6.3mm_D2.5mm_P2.54mm_Vertical
- gave numbers to parts that had none: 5
- renumbered Q5 to Q10, Q6 to Q11, Q7 to Q5, Q8 to Q6, Q9 to Q7, Q10 to Q8, Q11 to Q9, U8 to U10, U9 to U8, U10 to U9

Commit message: Simplify display driver board, add busy light
Removed digit storage and multiplexing logic from display driver, will handle in software instead
Add driver for busy indicator
Parts:
- renumbered Q9 to Q10, Q10 to Q11, Q11 to Q12, Q12 to Q13, Q13 to Q14, Q14 to Q15, Q15 to Q16, Q4 to Q5, Q5 to Q6, Q6 to Q7, Q7 to Q8, Q8 to Q9, R11 to R10, R12 to R11, R13 to R12, R14 to R13, R15 to R14, R16 to R15, R17 to R16, R6 to R5, R7 to R6, R8 to R7, R9 to R8, R10 to R9

Commit message: Display driver board routing and silkscreen tweaks
Parts:
- Q10, Q11, Q12, Q13, Q14, Q15, Q16, Q5, Q6, Q7, Q8, Q9: footprint Package_TO_SOT_THT:TO-92_Inline -> Package_TO_SOT_THT:TO-92_Inline_Wide
- R10, R11, R12, R13, R14, R15, R16, R5, R6, R7, R8, R9: footprint Resistor_THT:R_Axial_DIN0207_L6.3mm_D2.5mm_P2.54mm_Vertical -> Resistor_THT:R_Axial_DIN0207_L6.3mm_D2.5mm_P7.62mm_Horizontal
- renumbered U10 to U14
Connections:
- net ~{DP_0}: now also U10.9; no longer U10.11
- net ~{DP_10}: now also U14.13; no longer U14.5
- net ~{DP_11}: now also U14.11; no longer U14.9
- net ~{DP_1}: now also U10.5; no longer U10.13
- net ~{DP_2}: now also U10.3; no longer U10.1
- net ~{DP_3}: now also U10.1; no longer U10.3
- net ~{DP_4}: now also U11.13; no longer U11.5
- net ~{DP_5}: now also U11.11; no longer U11.9
- net ~{DP_6}: now also U11.9; no longer U11.11
- net ~{DP_7}: now also U11.5; no longer U11.13
- net ~{DP_8}: now also U11.3; no longer U11.1
- net ~{DP_9}: now also U11.1; no longer U11.3
- net at R12.1: now also U14.10; no longer U14.8
- net at U11.12: now also R9.1; no longer R14.1
- net at R13.1: now also U11.8; no longer U11.10
- net at R11.1: now also U14.12; no longer U14.6
- net at U10.2: now also R8.1; no longer R7.1
- net at R16.1: now also U11.2; no longer U11.4
- net at R5.1: now also U10.8; no longer U10.10
- net at U10.4: now also R7.1; no longer R8.1
- net at R10.1: now also U11.10; no longer U11.8
- net at R6.1: now also U10.6; no longer U10.12
- net at U11.6: now also R14.1; no longer R9.1
- net at R15.1: now also U11.4; no longer U11.2
Other:
- moved on the sheet: U10A, U10B, U11A, U11B, U11C, U11D, U11E, U11F

Commit message: Display driver geographical reannotate
Parts:
- renumbered Q7 to Q12, Q10 to Q13, Q15 to Q14, Q12 to Q15, Q5 to Q2, Q6 to Q25, Q9 to Q26, Q14 to Q27, Q11 to Q28, Q8 to Q3, Q13 to Q4, Q16 to Q5, R6 to R17, R8 to R18, R10 to R19, R14 to R20, R16 to R21, R12 to R22, R5 to R37, R7 to R38, R9 to R39, R13 to R40, R15 to R41, R11 to R42, U8 to U10, U9 to U11, U10 to U5, U11 to U6, U14 to U7

Commit message: Convert to KiCad 9.0
Convert to KiCad 9.0 format
Tweak silkscreen to fix DRC errors introduced by updated footprints
Changed lines of the file:
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@@
 (kicad_sch
-	(version 20231120)
+	(version 20250114)
 	(generator "eeschema")
-	(generator_version "8.0")
+	(generator_version "9.0")
 	(paper "USLetter")
 	(title_block
@@
 	(label "~{DP_4}"
 		(at 82.55 38.1 0)
-		(fields_autoplaced yes)
 		(effects
 			(font
@@
 	(label "~{DP_11}"
 		(at 168.91 152.4 180)
-		(fields_autoplaced yes)
 		(effects
 			(font
@@
 	(label "~{DP_4}"
 		(at 105.41 127 180)
-		(fields_autoplaced yes)
 		(effects
 			(font
@@
 	(label "~{DP_6}"
 		(at 170.18 25.4 180)
-		(fields_autoplaced yes)
 		(effects
 			(font
@@
 	(label "~{DP_8}"
 		(at 170.18 76.2 180)
-		(fields_autoplaced yes)
 		(effects
 			(font
@@
 	(label "~{DP_10}"
 		(at 168.91 127 180)
-		(fields_autoplaced yes)
 		(effects
 			(font
@@
 	(label "GND"
 		(at 57.15 45.72 180)
-		(fields_autoplaced yes)
 		(effects
 			(font
@@
 	(label "~{DP_6}"
 		(at 82.55 43.18 0)
-		(fields_autoplaced yes)
 		(effects
 			(font
@@
 	(label "~{DP_3}"
 		(at 82.55 35.56 0)
-		(fields_autoplaced yes)
 		(effects
 			(font
@@
 	(label "~{DP_0}"
 		(at 82.55 27.94 0)
-		(fields_autoplaced yes)
 		(effects
 			(font
@@
 	(label "~{DP_5}"
 		(at 105.41 152.4 180)
-		(fields_autoplaced yes)
 		(effects
 			(font
@@
 	(label "~{DP_2}"
 		(at 82.55 33.02 0)
-		(fields_autoplaced yes)
 		(effects
 			(font
@@
 	(label "~{DP_9}"
 		(at 170.18 101.6 180)
-		(fields_autoplaced yes)
 		(effects
 			(font
@@
 	(label "~{DP_1}"
 		(at 105.41 50.8 180)
-		(fields_autoplaced yes)
 		(effects
 			(font
@@
 	(label "~{DP_7}"
 		(at 170.18 50.8 180)
-		(fields_autoplaced yes)
 		(effects
 			(font
@@
 	(label "~{DP_[0..11]}"
 		(at 95.25 166.37 0)
-		(fields_autoplaced yes)
 		(effects
 			(font
@@
 	(label "~{DP_2}"
 		(at 105.41 76.2 180)
-		(fields_autoplaced yes)
 		(effects
 			(font
@@
 	(label "~{DP_0}"
 		(at 105.41 25.4 180)
-		(fields_autoplaced yes)
 		(effects
 			(font
@@
 	(label "~{DP_1}"
 		(at 82.55 30.48 0)
-		(fields_autoplaced yes)
 		(effects
 			(font
@@
 	(label "~{DP_3}"
 		(at 105.41 101.6 180)
-		(fields_autoplaced yes)
 		(effects
 			(font
@@
 	(label "~{DP_11}"
 		(at 82.55 83.82 0)
-		(fields_autoplaced yes)
 		(effects
 			(font
@@
 	(label "~{DP_7}"
 		(at 82.55 45.72 0)
-		(fields_autoplaced yes)
 		(effects
 			(font
@@
 	(label "VCC"
 		(at 57.15 40.64 180)
-		(fields_autoplaced yes)
 		(effects
 			(font
@@
 	(label "~{DP_9}"
 		(at 82.55 78.74 0)
-		(fields_autoplaced yes)
 		(effects
 			(font
@@
 	(label "GND"
 		(at 57.15 91.44 180)
-		(fields_autoplaced yes)
 		(effects
 			(font
@@
 	(label "~{DP_10}"
 		(at 82.55 81.28 0)
-		(fields_autoplaced yes)
 		(effects
 			(font
@@
 	(label "GND"
 		(at 57.15 93.98 180)
-		(fields_autoplaced yes)
 		(effects
 			(font
@@
 	(label "~{DP_5}"
 		(at 82.55 40.64 0)
-		(fields_autoplaced yes)
 		(effects
 			(font
@@
 	(label "~{DP_8}"
 		(at 82.55 76.2 0)
-		(fields_autoplaced yes)
 		(effects
 			(font
@@
 		(shape output)
 		(at 140.97 121.92 0)
-		(fields_autoplaced yes)
 		(effects
 			(font
@@
 		(shape output)
 		(at 140.97 45.72 0)
-		(fields_autoplaced yes)
 		(effects
 			(font
@@
 		(shape input)
 		(at 38.1 30.48 180)
-		(fields_autoplaced yes)
 		(effects
 			(font
@@
 		(shape output)
 		(at 205.74 71.12 0)
-		(fields_autoplaced yes)
 		(effects
 			(font
@@
 		(shape output)
 		(at 204.47 121.92 0)
-		(fields_autoplaced yes)
 		(effects
 			(font
@@
 		(shape output)
 		(at 205.74 45.72 0)
-		(fields_autoplaced yes)
 		(effects
 			(font
@@
 		(shape output)
 		(at 140.97 147.32 0)
-		(fields_autoplaced yes)
 		(effects
 			(font
@@
 		(shape input)
 		(at 38.1 33.02 180)
-		(fields_autoplaced yes)
 		(effects
 			(font
@@
 		(shape output)
 		(at 204.47 147.32 0)
-		(fields_autoplaced yes)
 		(effects
 			(font
@@
 		(shape input)
 		(at 38.1 35.56 180)
-		(fields_autoplaced yes)
 		(effects
 			(font
@@
 		(shape output)
 		(at 205.74 20.32 0)
-		(fields_autoplaced yes)
 		(effects
 			(font
@@
 		(shape output)
 		(at 140.97 20.32 0)
-		(fields_autoplaced yes)
 		(effects
 			(font
@@
 		(shape output)
 		(at 205.74 96.52 0)
-		(fields_autoplaced yes)
 		(effects
 			(font
@@
 		(shape output)
 		(at 140.97 96.52 0)
-		(fields_autoplaced yes)
 		(effects
 			(font
@@
 		(shape output)
 		(at 140.97 71.12 0)
-		(fields_autoplaced yes)
 		(effects
 			(font
@@
 		(shape input)
 		(at 38.1 27.94 180)
-		(fields_autoplaced yes)
-		(effects
-			(font
+		(effects
+			(font

Commit message: Minor display hardware revisions
Add anti-ghosting inter-cathode resistors to nixies
Adjust component values based on experiments
Change from individual netclass labels to rule areas
Tweak traces on display board
Update .gitignore to ignore KiCad lock files
Parts:
- R17, R18, R19, R20, R21, R22, R37, R38, R39, R40, R41, R42: value 1k -> 10k
Changed lines of the file:
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@@
 			)
 		)
-		(property "Value" "1k"
+		(property "Value" "10k"
 			(at 190.5 21.59 90)
 			(effects
@@
 			)
 		)
-		(property "Value" "1k"
+		(property "Value" "10k"
 			(at 190.5 97.79 90)
 			(effects
@@
 			)
 		)
-		(property "Value" "1k"
+		(property "Value" "10k"
 			(at 125.73 21.59 90)
 			(effects
@@
 			)
 		)
-		(property "Value" "1k"
+		(property "Value" "10k"
 			(at 125.73 72.39 90)
 			(effects
@@
 			)
 		)
-		(property "Value" "1k"
+		(property "Value" "10k"
 			(at 189.23 148.59 90)
 			(effects
@@
 			)
 		)
-		(property "Value" "1k"
+		(property "Value" "10k"
 			(at 125.73 123.19 90)
 			(effects
@@
 			)
 		)
-		(property "Value" "1k"
+		(property "Value" "10k"
 			(at 190.5 72.39 90)
 			(effects
@@
 			)
 		)
-		(property "Value" "1k"
+		(property "Value" "10k"
 			(at 189.23 123.19 90)
 			(effects
@@
 			)
 		)
-		(property "Value" "1k"
+		(property "Value" "10k"
 			(at 190.5 46.99 90)
 			(effects
@@
 			)
 		)
-		(property "Value" "1k"
+		(property "Value" "10k"
 			(at 125.73 148.59 90)
 			(effects
@@
 			)
 		)
-		(property "Value" "1k"
+		(property "Value" "10k"
 			(at 125.73 46.99 90)
 			(effects
@@
 			)
 		)
-		(property "Value" "1k"
+		(property "Value" "10k"
 			(at 125.73 97.79 90)
 			(effects
